File: Ecardz-Proto/Ecardz-Proto.kicad_pcb (KiCad board)
At the start: 4 copper layers, 110 x 90 mm, 75 parts, among them IC1 M24LR04E-RMN6T/2, J1 Conn_02x06_Odd_Even, J2 Conn_01x24, J3 Conn_ARM_SWD_TagConnect_TC203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, J4 Conn_02x07_Odd_Even, Q1 NMOS, U1 STM32L071K8Ux

Commit message: silkscreen images
and fixed layout DRCs
Routing:
- net /NFC/V_E_HARVEST: track 34.5 -> 50.2 mm
- net /STM/I2C_NFC_SDA: track 16.6 -> 23.6 mm
- net VDD: track 230.0 -> 234.6 mm, vias 11 -> 12
- net GND: track 33.5 -> 32.2 mm, vias 28 -> 41
- net /STM/NFC_BUSY: track 61.0 -> 60.4 mm
Other:
- board text added: "E-Card Rev 1 Avi Cahoon Isabella Schneider"
- board text added: "SPI3"
- board text added: "SPI4"

Commit message: gerbers generated for first fab
Routing:
- net GND: track 32.2 -> 33.4 mm, vias 41 -> 40

Commit message: added stitching vias
Routing:
- net GND: vias 40 -> 121
