File: Ecardz-Controller/Ecardz-Controller.kicad_pcb (KiCad board)
At the start: 2 copper layers, 0 parts

Commit message: initial work on controller layout
Parts:
- added C1: 8.2p, Capacitor_SMD:C_0603_1608Metric_Pad1.08x0.95mm_HandSolder, F.Cu at (193.2, 99.6)
- added C10: 10n, Capacitor_SMD:C_0603_1608Metric_Pad1.08x0.95mm_HandSolder, F.Cu at (197.3, 105.9)
- added C11: 2.2u, Capacitor_SMD:C_0603_1608Metric_Pad1.08x0.95mm_HandSolder, F.Cu at (200.6, 111.4)
- added C12: 2.2u, Capacitor_SMD:C_0603_1608Metric_Pad1.08x0.95mm_HandSolder, F.Cu at (197.4, 108.9)
- added C13: 10n, Capacitor_SMD:C_0603_1608Metric_Pad1.08x0.95mm_HandSolder, F.Cu at (202.1, 111.4)
- added C14: 10n, Capacitor_SMD:C_0603_1608Metric_Pad1.08x0.95mm_HandSolder, F.Cu at (197.4, 107.4)
- added C15: 2.2u, Capacitor_SMD:C_0603_1608Metric_Pad1.08x0.95mm_HandSolder, F.Cu at (203.6, 111.4)
- added C16: 22n, Capacitor_SMD:C_0603_1608Metric_Pad1.08x0.95mm_HandSolder, F.Cu at (205.1, 111.4)
- added C17: 1uF, Capacitor_SMD:C_0603_1608Metric_Pad1.08x0.95mm_HandSolder, F.Cu at (208.4, 101.6)
- added C18: 10n, Capacitor_SMD:C_0603_1608Metric_Pad1.08x0.95mm_HandSolder, F.Cu at (208.4, 100.1)
- added C19: 100nF, Capacitor_SMD:C_0603_1608Metric_Pad1.08x0.95mm_HandSolder, B.Cu at (112.1, 142.8)
- added C2: 1uF, Capacitor_SMD:C_0603_1608Metric_Pad1.08x0.95mm_HandSolder, F.Cu at (202.2, 98.1)
- added C20: 1uF, Capacitor_SMD:C_0603_1608Metric_Pad1.08x0.95mm_HandSolder, B.Cu at (112.1, 141.2)
- added C21: 100nF, Capacitor_SMD:C_0603_1608Metric_Pad1.08x0.95mm_HandSolder, B.Cu at (112.1, 145.9)
- added C22: 4.7uF, Capacitor_SMD:C_0603_1608Metric_Pad1.08x0.95mm_HandSolder, B.Cu at (112.1, 144.2)
- added C23: 1uF, Capacitor_SMD:C_0603_1608Metric_Pad1.08x0.95mm_HandSolder, F.Cu at (257.1, 119.6)
- added C24: 1uF, Capacitor_SMD:C_0603_1608Metric_Pad1.08x0.95mm_HandSolder, F.Cu at (257.1, 122.1)
- added C25: 1uF, Capacitor_SMD:C_0603_1608Metric_Pad1.08x0.95mm_HandSolder, F.Cu at (257.1, 124.6)
- added C26: DNP, Capacitor_SMD:C_0603_1608Metric_Pad1.08x0.95mm_HandSolder, F.Cu at (257.1, 127.1)
- added C27: 1uF, Capacitor_SMD:C_0603_1608Metric_Pad1.08x0.95mm_HandSolder, F.Cu at (257.1, 129.6)
- added C28: 1uF, Capacitor_SMD:C_0603_1608Metric_Pad1.08x0.95mm_HandSolder, F.Cu at (257.1, 132.1)
- added C29: 1uF, Capacitor_SMD:C_0603_1608Metric_Pad1.08x0.95mm_HandSolder, F.Cu at (257.1, 134.6)
- added C3: 8.2p, Capacitor_SMD:C_0603_1608Metric_Pad1.08x0.95mm_HandSolder, F.Cu at (191.8, 107.1)
- added C30: 1uF, Capacitor_SMD:C_0603_1608Metric_Pad1.08x0.95mm_HandSolder, F.Cu at (257.1, 137.2)
- added C31: 1uF, Capacitor_SMD:C_0603_1608Metric_Pad1.08x0.95mm_HandSolder, F.Cu at (261.5, 119.6)
- added C32: 1uF, Capacitor_SMD:C_0603_1608Metric_Pad1.08x0.95mm_HandSolder, F.Cu at (261.5, 122.1)
- added C33: 10uF, Capacitor_SMD:C_0805_2012Metric_Pad1.18x1.45mm_HandSolder, F.Cu at (329.1, 85.6)
- added C34: 22uF, Capacitor_SMD:C_0805_2012Metric_Pad1.18x1.45mm_HandSolder, F.Cu at (329.1, 88.6)
- added C35: 1uF, Capacitor_SMD:C_0603_1608Metric_Pad1.08x0.95mm_HandSolder, F.Cu at (324.6, 85.4)
- added C36: 1uF, Capacitor_SMD:C_0603_1608Metric_Pad1.08x0.95mm_HandSolder, F.Cu at (324.6, 87.9)
- added C37: 100nF, Capacitor_SMD:C_0603_1608Metric_Pad1.08x0.95mm_HandSolder, B.Cu at (79.9, 182.7)
- added C38: 1uF, Capacitor_SMD:C_0603_1608Metric_Pad1.08x0.95mm_HandSolder, B.Cu at (79.9, 185.2)
- added C39: 4.7uF, Capacitor_SMD:C_0603_1608Metric_Pad1.08x0.95mm_HandSolder, B.Cu at (78.9, 136.0)
- added C4: 100n, Capacitor_SMD:C_0603_1608Metric_Pad1.08x0.95mm_HandSolder, F.Cu at (200.8, 98.1)
- added C40: 4.7uF, Capacitor_SMD:C_0603_1608Metric_Pad1.08x0.95mm_HandSolder, B.Cu at (88.9, 137.0)
- added C41: 100nF, Capacitor_SMD:C_0603_1608Metric_Pad1.08x0.95mm_HandSolder, B.Cu at (88.9, 135.5)
- added C42: LXRW0YV600-054, samacsys:LXRW0YV600054, F.Cu at (208.9, 130.5)
- added C43: LXRW0YV600-054, samacsys:LXRW0YV600054, F.Cu at (208.9, 133.2)
- added C44: LXRW0YV600-054, samacsys:LXRW0YV600054, F.Cu at (208.9, 135.9)
- added C45: 680pF, Capacitor_SMD:C_0603_1608Metric_Pad1.08x0.95mm_HandSolder, F.Cu at (213.2, 129.5)
- added C46: 680pF, Capacitor_SMD:C_0603_1608Metric_Pad1.08x0.95mm_HandSolder, F.Cu at (213.2, 132.0)
- added C47: 180pF, Capacitor_SMD:C_0603_1608Metric_Pad1.08x0.95mm_HandSolder, F.Cu at (213.2, 134.5)
- added C48: 180pF, Capacitor_SMD:C_0603_1608Metric_Pad1.08x0.95mm_HandSolder, F.Cu at (213.2, 137.0)
- added C49: 82pF, Capacitor_SMD:C_0603_1608Metric_Pad1.08x0.95mm_HandSolder, F.Cu at (213.2, 139.5)
- added C5: 2.2u, Capacitor_SMD:C_0603_1608Metric_Pad1.08x0.95mm_HandSolder, F.Cu at (198.0, 100.1)
- added C50: 10pF, Capacitor_SMD:C_0603_1608Metric_Pad1.08x0.95mm_HandSolder, F.Cu at (213.2, 142.0)
- added C51: 10pF, Capacitor_SMD:C_0603_1608Metric_Pad1.08x0.95mm_HandSolder, F.Cu at (217.6, 129.5)
- added C52: 82pF, Capacitor_SMD:C_0603_1608Metric_Pad1.08x0.95mm_HandSolder, F.Cu at (217.6, 132.0)
- added C53: 240pF, Capacitor_SMD:C_0603_1608Metric_Pad1.08x0.95mm_HandSolder, F.Cu at (217.6, 134.5)
- added C6: 2.2u, Capacitor_SMD:C_0603_1608Metric_Pad1.08x0.95mm_HandSolder, F.Cu at (197.6, 111.4)
- added C7: 10n, Capacitor_SMD:C_0603_1608Metric_Pad1.08x0.95mm_HandSolder, F.Cu at (198.0, 101.6)
- added C8: 10n, Capacitor_SMD:C_0603_1608Metric_Pad1.08x0.95mm_HandSolder, F.Cu at (199.1, 111.4)
- added C9: 2.2u, Capacitor_SMD:C_0603_1608Metric_Pad1.08x0.95mm_HandSolder, F.Cu at (197.3, 104.4)
- added D1: LED-G, LED_SMD:LED_0603_1608Metric_Pad1.05x0.95mm_HandSolder, F.Cu at (109.8, 95.6)
- added D10: D_Schottky, Diode_SMD:D_SOD-123, B.Cu at (105.6, 175.7)
- added D11: D_Schottky, Diode_SMD:D_SOD-123, B.Cu at (105.6, 179.0)
- added D12: RB521S30T1G, Diode_SMD:D_SOD-523, F.Cu at (328.6, 96.0)
- added D13: RB521S30T1G, Diode_SMD:D_SOD-523, F.Cu at (328.6, 98.4)
- added D2: LED-R, LED_SMD:LED_0603_1608Metric_Pad1.05x0.95mm_HandSolder, F.Cu at (112.4, 95.6)
- added D3: LED-B, LED_SMD:LED_0603_1608Metric_Pad1.05x0.95mm_HandSolder, F.Cu at (115.0, 95.6)
- added D4: LED-B, LED_SMD:LED_0603_1608Metric_Pad1.05x0.95mm_HandSolder, F.Cu at (98.8, 126.5)
- added D5: LED-R, LED_SMD:LED_0603_1608Metric_Pad1.05x0.95mm_HandSolder, F.Cu at (106.0, 126.5)
- added D6: LED-G, LED_SMD:LED_0603_1608Metric_Pad1.05x0.95mm_HandSolder, F.Cu at (113.0, 126.5)
- added D7: LED-G, LED_SMD:LED_0603_1608Metric_Pad1.05x0.95mm_HandSolder, F.Cu at (52.7, 130.9)
- added D8: LED-G, LED_SMD:LED_0603_1608Metric_Pad1.05x0.95mm_HandSolder, F.Cu at (58.8, 130.9)
- added D9: D_Schottky, Diode_SMD:D_SOD-123, B.Cu at (105.6, 172.3)
- added IC1: ST25R3916B-AQWT, samacsys:QFN50P500X500X100-33N-D, F.Cu at (203.4, 103.6)
- added J1: MEM2061-01-188-00-A, samacsys:MEM20610118800A, F.Cu at (57.9, 113.2)
- added J6: Conn_01x24, Connector_FFC-FPC:TE_2-1734839-4_1x24-1MP_P0.5mm_Horizontal, B.Cu at (67.3, 180.2)
- added J7: Conn_01x02, Connector_PinHeader_2.54mm:PinHeader_1x02_P2.54mm_Vertical, F.Cu at (99.2, 94.0)
- added L1: L, parts-lib:CDRH5D18, B.Cu at (89.0, 179.0)
- added L3: 270nH, parts-lib:CDRH5D18, F.Cu at (209.1, 111.9)
- added L4: 270nH, parts-lib:CDRH5D18, F.Cu at (215.9, 111.9)
- added LS1: PS1240P02BT, samacsys:PS1240P02BT, F.Cu at (80.0, 99.0)
- added Q1: NMOS, Package_TO_SOT_SMD:SOT-23, B.Cu at (94.5, 178.0)
- added R1: .5R, Resistor_SMD:R_0603_1608Metric_Pad0.98x0.95mm_HandSolder, F.Cu at (209.0, 107.6)
- added R10: 10k, Resistor_SMD:R_0603_1608Metric_Pad0.98x0.95mm_HandSolder, F.Cu at (108.0, 126.4)
- added R11: 10k, Resistor_SMD:R_0603_1608Metric_Pad0.98x0.95mm_HandSolder, F.Cu at (115.0, 126.4)
- added R12: 4.7k, Resistor_SMD:R_0603_1608Metric_Pad0.98x0.95mm_HandSolder, B.Cu at (104.3, 135.5)
- added R13: 4.7k, Resistor_SMD:R_0603_1608Metric_Pad0.98x0.95mm_HandSolder, B.Cu at (102.8, 135.5)
- added R14: 10k, Resistor_SMD:R_0603_1608Metric_Pad0.98x0.95mm_HandSolder, F.Cu at (52.8, 134.9)
- added R15: 10k, Resistor_SMD:R_0603_1608Metric_Pad0.98x0.95mm_HandSolder, F.Cu at (58.8, 134.9)
- added R16: 4.7k, Resistor_SMD:R_0603_1608Metric_Pad0.98x0.95mm_HandSolder, B.Cu at (107.4, 135.5)
- added R17: 4.7k, Resistor_SMD:R_0603_1608Metric_Pad0.98x0.95mm_HandSolder, B.Cu at (105.8, 135.5)
- added R18: 1k, Resistor_SMD:R_0603_1608Metric_Pad0.98x0.95mm_HandSolder, F.Cu at (261.5, 124.6)
- added R19: 10k, Resistor_SMD:R_0603_1608Metric_Pad0.98x0.95mm_HandSolder, F.Cu at (261.5, 127.1)
- added R2: 0, Resistor_SMD:R_0603_1608Metric_Pad0.98x0.95mm_HandSolder, F.Cu at (205.4, 95.2)
- added R20: 10k, Resistor_SMD:R_0603_1608Metric_Pad0.98x0.95mm_HandSolder, F.Cu at (261.5, 129.6)
- added R21: 10k, Resistor_SMD:R_0603_1608Metric_Pad0.98x0.95mm_HandSolder, F.Cu at (261.5, 132.1)
- added R22: 10k, Resistor_SMD:R_0603_1608Metric_Pad0.98x0.95mm_HandSolder, F.Cu at (261.5, 134.6)
- added R23: 10k, Resistor_SMD:R_0603_1608Metric_Pad0.98x0.95mm_HandSolder, F.Cu at (261.5, 137.2)
- added R24: 10k, Resistor_SMD:R_0603_1608Metric_Pad0.98x0.95mm_HandSolder, F.Cu at (265.8, 119.6)
- added R25: 10k, Resistor_SMD:R_0603_1608Metric_Pad0.98x0.95mm_HandSolder, F.Cu at (265.8, 122.1)
- added R26: 2.2R, Resistor_SMD:R_0603_1608Metric_Pad0.98x0.95mm_HandSolder, F.Cu at (265.8, 124.6)
- added R27: DNP, Resistor_SMD:R_0603_1608Metric_Pad0.98x0.95mm_HandSolder, B.Cu at (73.3, 185.8)
- added R28: 0R, Resistor_SMD:R_0603_1608Metric_Pad0.98x0.95mm_HandSolder, B.Cu at (73.3, 181.0)
- added R29: 0R, Resistor_SMD:R_0603_1608Metric_Pad0.98x0.95mm_HandSolder, B.Cu at (73.3, 182.5)
- added R3: 0, Resistor_SMD:R_0603_1608Metric_Pad0.98x0.95mm_HandSolder, F.Cu at (203.8, 95.2)
- added R31: 800k, Resistor_SMD:R_0603_1608Metric_Pad0.98x0.95mm_HandSolder, F.Cu at (324.6, 90.4)
- added R32: 200k, Resistor_SMD:R_0603_1608Metric_Pad0.98x0.95mm_HandSolder, F.Cu at (324.6, 92.9)
- added R34: DNP, Resistor_SMD:R_0603_1608Metric_Pad0.98x0.95mm_HandSolder, F.Cu at (324.6, 95.4)
- added R35: 0R, Resistor_SMD:R_0603_1608Metric_Pad0.98x0.95mm_HandSolder, F.Cu at (324.6, 97.9)
- added R36: DNP, Resistor_SMD:R_0603_1608Metric_Pad0.98x0.95mm_HandSolder, F.Cu at (324.6, 100.4)
- added R37: 0R, Resistor_SMD:R_0603_1608Metric_Pad0.98x0.95mm_HandSolder, F.Cu at (324.6, 103.0)
- added R38: 0R, Resistor_SMD:R_0603_1608Metric_Pad0.98x0.95mm_HandSolder, F.Cu at (319.5, 120.1)
- added R39: 0R, Resistor_SMD:R_0603_1608Metric_Pad0.98x0.95mm_HandSolder, F.Cu at (319.5, 122.6)
- added R4: 0, Resistor_SMD:R_0603_1608Metric_Pad0.98x0.95mm_HandSolder, F.Cu at (228.8, 114.5)
- added R40: 0, Resistor_SMD:R_0603_1608Metric_Pad0.98x0.95mm_HandSolder, F.Cu at (233.2, 123.8)
- added R41: 0, Resistor_SMD:R_0603_1608Metric_Pad0.98x0.95mm_HandSolder, F.Cu at (233.2, 126.3)
- added R42: 0, Resistor_SMD:R_0603_1608Metric_Pad0.98x0.95mm_HandSolder, F.Cu at (233.2, 128.8)
- added R43: 0, Resistor_SMD:R_0603_1608Metric_Pad0.98x0.95mm_HandSolder, F.Cu at (227.8, 124.2)
- added R44: 0, Resistor_SMD:R_0603_1608Metric_Pad0.98x0.95mm_HandSolder, F.Cu at (227.8, 126.7)
- added R45: 0, Resistor_SMD:R_0603_1608Metric_Pad0.98x0.95mm_HandSolder, F.Cu at (227.8, 129.2)
- added R46: 0, Resistor_SMD:R_0603_1608Metric_Pad0.98x0.95mm_HandSolder, F.Cu at (227.8, 131.8)
- added R5: 0, Resistor_SMD:R_0603_1608Metric_Pad0.98x0.95mm_HandSolder, F.Cu at (229.6, 117.8)
- added R6: 10k, Resistor_SMD:R_0603_1608Metric_Pad0.98x0.95mm_HandSolder, F.Cu at (109.9, 99.4)
- added R7: 10k, Resistor_SMD:R_0603_1608Metric_Pad0.98x0.95mm_HandSolder, F.Cu at (112.5, 99.4)
- added R8: 10k, Resistor_SMD:R_0603_1608Metric_Pad0.98x0.95mm_HandSolder, F.Cu at (115.0, 99.5)
- added R9: 10k, Resistor_SMD:R_0603_1608Metric_Pad0.98x0.95mm_HandSolder, F.Cu at (100.8, 126.4)
- added REF**: MountingHole_2.7mm_M2.5_Pad_TopBottom, MountingHole:MountingHole_2.7mm_M2.5_Pad_TopBottom, F.Cu at (84.0, 195.0)
- added REF**: MountingHole_2.7mm_M2.5_Pad_TopBottom, MountingHole:MountingHole_2.7mm_M2.5_Pad_TopBottom, F.Cu at (84.0, 148.0)
- added REF**: MountingHole_2.7mm_M2.5_Pad_TopBottom, MountingHole:MountingHole_2.7mm_M2.5_Pad_TopBottom, F.Cu at (176.0, 195.0)
- added REF**: MountingHole_2.7mm_M2.5_Pad_TopBottom, MountingHole:MountingHole_2.7mm_M2.5_Pad_TopBottom, F.Cu at (176.0, 148.0)
- added S1: PRT-14460, samacsys:PRT14460, F.Cu at (104.2, 106.8)
- added S2: PRT-14460, samacsys:PRT14460, F.Cu at (87.8, 115.5)
- added S3: PRT-14460, samacsys:PRT14460, F.Cu at (162.5, 97.1)
- added S4: PRT-14460, samacsys:PRT14460, F.Cu at (148.0, 111.0)
- added S5: PRT-14460, samacsys:PRT14460, F.Cu at (177.0, 111.0)
- added S6: PRT-14460, samacsys:PRT14460, F.Cu at (162.5, 125.5)
- added S7: PRT-14460, samacsys:PRT14460, F.Cu at (62.0, 94.0)
- added TP1: TestPoint, TestPoint:TestPoint_Pad_1.0x1.0mm, F.Cu at (198.8, 98.2)
- added TP2: TestPoint, TestPoint:TestPoint_Pad_1.0x1.0mm, F.Cu at (204.8, 98.5)
- added TP3: TestPoint, TestPoint:TestPoint_Pad_1.0x1.0mm, F.Cu at (66.0, 135.5)
- added TP4: TestPoint, TestPoint:TestPoint_Pad_D3.0mm, F.Cu at (124.8, 95.5)
- added TP5: TestPoint, TestPoint:TestPoint_Pad_D3.0mm, F.Cu at (129.9, 95.5)
- added TP6: TestPoint, TestPoint:TestPoint_Pad_D3.0mm, F.Cu at (134.9, 95.5)
- added TP7: TestPoint, TestPoint:TestPoint_Pad_D3.0mm, F.Cu at (140.0, 95.5)
- added TP8: TestPoint, TestPoint:TestPoint_Pad_D3.0mm, F.Cu at (188.0, 94.0)
- added TP9: TestPoint, TestPoint:TestPoint_Pad_D3.0mm, F.Cu at (188.0, 99.0)
- added U1: STM32G0C1RETx, Package_QFP:LQFP-64_10x10mm_P0.5mm, B.Cu at (103.3, 144.0)
- added U2: TPS62160DSG, Package_SON:WSON-8-1EP_2x2mm_P0.5mm_EP0.9x1.6mm_ThermalVias, F.Cu at (125.8, 117.8)
- added U3: MIC5504-3.3YM5, Package_TO_SOT_SMD:SOT-23-5, F.Cu at (329.3, 92.5)
- added U4: CP2110-F02-GM1, Package_DFN_QFN:QFN-28-1EP_5x5mm_P0.5mm_EP3.35x3.35mm, B.Cu at (83.9, 136.0)
- added Y1: XRCGB27M120F3M00R0, samacsys:XRCGB, F.Cu at (193.4, 103.4)
Routing:
- net /MCU/NFC_BUSY: track 0.00 -> 140.5 mm, vias 0 -> 1
- net +3V3: track 0.00 -> 26.4 mm, vias 0 -> 1
- net GND: track 0.00 -> 13.9 mm, vias 0 -> 2
- net /NFC/ANTENNA/RFO2: track 0.00 -> 13.3 mm
- net /MCU/NFC_I_SENSE: track 0.00 -> 12.2 mm
- net Net-(IC1-XTI): track 0.00 -> 12.2 mm
- net Net-(IC1-XTO): track 0.00 -> 10.0 mm
- net /INTERFACE/BS1: track 0.00 -> 8.03 mm
- net /NFC/ANTENNA/RFO1: track 0.00 -> 7.78 mm
- net Net-(IC1-BSS): track 0.00 -> 6.93 mm
- net /INTERFACE/GDR: track 0.00 -> 6.53 mm
- net Net-(IC1-VDD_AM): track 0.00 -> 6.36 mm
- net Net-(IC1-TAD2): track 0.00 -> 5.52 mm
- net Net-(IC1-VDD_A): track 0.00 -> 4.52 mm
- net Net-(IC1-VDD_D): track 0.00 -> 3.96 mm
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Other:
- board outline added: 189 x 115 mm
- copper layers 2 -> 4
- board text removed: "DSIU 01-06-2025"
- board text removed: "For Instructional Use Only."
- board text removed: "SOLIDWORKS Educational Product."

Commit message: did bulk of controller layout apart from the antenna, added some NCs and other minor clean ups on schematic
Parts:
- removed REF** (x4): MountingHole_2.7mm_M2.5_Pad_TopBottom, MountingHole:MountingHole_2.7mm_M2.5_Pad_TopBottom
- added H1: MountingHole_Pad, MountingHole:MountingHole_2.7mm_M2.5_Pad_TopBottom, F.Cu at (60.0, 100.0)
- added H2: MountingHole_Pad, MountingHole:MountingHole_2.7mm_M2.5_Pad_TopBottom, F.Cu at (229.0, 100.0)
- added H3: MountingHole_Pad, MountingHole:MountingHole_2.7mm_M2.5_Pad_TopBottom, F.Cu at (60.0, 195.0)
- added H4: MountingHole_Pad, MountingHole:MountingHole_2.7mm_M2.5_Pad_TopBottom, F.Cu at (229.0, 195.0)
- added H5: MountingHole_Pad, MountingHole:MountingHole_2.7mm_M2.5_Pad_TopBottom, F.Cu at (84.0, 148.0)
- added H6: MountingHole_Pad, MountingHole:MountingHole_2.7mm_M2.5_Pad_TopBottom, F.Cu at (176.0, 148.0)
- added H7: MountingHole_Pad, MountingHole:MountingHole_2.7mm_M2.5_Pad_TopBottom, F.Cu at (84.0, 195.0)
- added H8: MountingHole_Pad, MountingHole:MountingHole_2.7mm_M2.5_Pad_TopBottom, F.Cu at (176.0, 195.0)
- added J2: Conn_01x04, Connector_PinHeader_2.54mm:PinHeader_1x04_P2.54mm_Vertical, F.Cu at (104.8, 101.8)
- added J3: Conn_01x05, Connector_PinHeader_2.54mm:PinHeader_1x05_P2.54mm_Vertical, F.Cu at (187.0, 115.5)
- added J4: Conn_01x09, Connector_PinHeader_2.54mm:PinHeader_1x09_P2.54mm_Vertical, F.Cu at (59.2, 161.2)
- added J5: Conn_01x01, Connector_PinHeader_2.54mm:PinHeader_1x01_P2.54mm_Vertical, F.Cu at (59.2, 185.5)
- added J8: Conn_01x04, Connector_PinHeader_2.54mm:PinHeader_1x04_P2.54mm_Vertical, F.Cu at (62.2, 136.8)
- added L2: 2.2uH, samacsys:VLS2016, B.Cu at (99.1, 142.8)
- added R30: 100k, Resistor_SMD:R_0603_1608Metric_Pad0.98x0.95mm_HandSolder, B.Cu at (106.0, 139.9)
- added R33: 100k, Resistor_SMD:R_0603_1608Metric_Pad0.98x0.95mm_HandSolder, B.Cu at (99.6, 139.8)
- C1, C10, C11, C12, C13, C14, C15, C16, C17, C18, C2, C23, C24, C25, C26, C27, C28, C29, C3, C30, C31, C32, C33, C34, C35, C36, C4, C42, C43, C44, C45, C46, C47, C48, C49, C5, C50, C51, C52, C53, C6, C7, C8, C9, D1, D12, D13, D2, D3, D4, IC1, L3, L4, R1, R18, R19, R2, R20, R21, R22, R23, R24, R25, R26, R3, R31, R32, R34, R35, R36, R37, R38, R39, R4, R40, R41, R42, R43, R44, R45, R46, R5, R6, R7, R8, R9, U2, U3, Y1: moved to B.Cu
- TP1, TP2: footprint TestPoint:TestPoint_Pad_1.0x1.0mm -> TestPoint:TestPoint_Pad_D3.0mm; moved to B.Cu
- TP3: footprint TestPoint:TestPoint_Pad_1.0x1.0mm -> TestPoint:TestPoint_Pad_D3.0mm
- moved C33 259.1 mm to (74.0, 131.0)
- moved D12 257.9 mm to (73.3, 132.8), turned to 180 degrees
- moved D13 257.8 mm to (73.3, 134.2), turned to 180 degrees
- moved C34 237.5 mm to (98.7, 146.0), turned to 180 degrees
- moved R34 235.5 mm to (93.8, 142.1), turned to -90 degrees
- moved R35 233.3 mm to (95.5, 142.1), turned to 90 degrees
- moved R38 230.7 mm to (89.2, 134.0)
- moved R39 230.5 mm to (89.2, 132.5)
- moved C35 230.4 mm to (99.6, 134.8), turned to 180 degrees
- moved U3 229.4 mm to (103.6, 133.5)
- moved R31 228.4 mm to (102.2, 142.9), turned to 90 degrees
- moved R36 228.1 mm to (99.6, 137.8)
- moved R37 227.4 mm to (99.6, 136.2)
- moved C36 226.5 mm to (103.4, 136.5), turned to 180 degrees
- moved R32 226.4 mm to (103.8, 142.9), turned to -90 degrees
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Connections:
- IC1 pad 18: unconnected-(IC1-AAT_A-Pad18) -> /NFC/ANTENNA/AAT_A
- IC1 pad 19: unconnected-(IC1-AAT_B-Pad19) -> /NFC/ANTENNA/AAT_B
- R19 pad 1: /INTERFACE/BUTTON7 -> /INTERFACE/BUTTON1
- R20 pad 1: /INTERFACE/BUTTON6 -> /INTERFACE/BUTTON2
- R21 pad 1: /INTERFACE/BUTTON5 -> /INTERFACE/BUTTON3
- R23 pad 1: /INTERFACE/BUTTON3 -> /INTERFACE/BUTTON5
- R24 pad 1: /INTERFACE/BUTTON2 -> /INTERFACE/BUTTON6
- R25 pad 1: /INTERFACE/BUTTON1 -> /INTERFACE/BUTTON7
- S1 pad 2: /INTERFACE/BUTTON7 -> /INTERFACE/BUTTON1
- S2 pad 2: /INTERFACE/BUTTON6 -> /INTERFACE/BUTTON2
- S3 pad 2: /INTERFACE/BUTTON5 -> /INTERFACE/BUTTON3
- S5 pad 2: /INTERFACE/BUTTON3 -> /INTERFACE/BUTTON5
- S6 pad 2: /INTERFACE/BUTTON2 -> /INTERFACE/BUTTON6
- S7 pad 1: /INTERFACE/BUTTON1 -> unconnected-(S7-Pad1)
- S7 pad 2: unconnected-(S7-Pad2) -> /INTERFACE/BUTTON7
- U1 pad 21: /MCU/SD_CS -> /MCU/SPI_LCD_CS
- U1 pad 22: /MCU/EINK_SCK -> /MCU/SPI_LCD_SCK
- U1 pad 23: /MCU/EINK_MISO -> /MCU/SPI_LCD_MISO
- U1 pad 24: /MCU/EINK_MOSI -> /MCU/SPI_LCD_MOSI
- U1 pad 27: /INTERFACE/SPI_LCD_CS -> /MCU/SPI_LCD_CS
- U1 pad 28: /MCU/LCD_PWM_BRIGHT -> /INTERFACE/LCD_PWM_BRIGHT
- U1 pad 29: /MCU/SPI_LCD_DC -> /INTERFACE/SPI_LCD_DC
- U1 pad 36: /MCU/BUTTON7 -> /INTERFACE/BUTTON7
- U1 pad 37: /MCU/BUTTON6 -> /INTERFACE/BUTTON6
- U1 pad 38: /MCU/BUTTON5 -> /INTERFACE/BUTTON5
- U1 pad 39: /MCU/BUTTON4 -> /INTERFACE/BUTTON4
- U1 pad 42: /MCU/BUTTON3 -> /INTERFACE/BUTTON3
- U1 pad 43: /MCU/BUTTON2 -> /INTERFACE/BUTTON2
- U1 pad 44: /MCU/BUTTON1 -> /INTERFACE/BUTTON1
Routing:
- net /MCU/NFC_I_SENSE: track 12.2 -> 135.8 mm, vias 0 -> 3
- net /MCU/I2C_NFC_SDA: track 3.20 -> 122.6 mm, vias 1 -> 2
- net /MCU/I2C_NFC_SCL: track 2.99 -> 117.3 mm, vias 1 -> 2
- net GND: track 13.9 -> 119.1 mm, vias 2 -> 75
- net /MCU/SD_MOSI: track 0.00 -> 100.0 mm, vias 0 -> 1
- net /MCU/SD_MISO: track 0.00 -> 95.7 mm, vias 0 -> 1
- net /MCU/SD_SCK: track 0.00 -> 91.9 mm, vias 0 -> 1
- net /MCU/SPI_LCD_MISO: track 0.00 -> 79.6 mm, vias 0 -> 1
- net /INTERFACE/LCD_PWM_BRIGHT: track 0.00 -> 79.5 mm
- net /INTERFACE/CS#: track 0.00 -> 79.0 mm, vias 0 -> 2
- net /INTERFACE/D/C#: track 0.00 -> 78.6 mm, vias 0 -> 2
- net /INTERFACE/SCL: track 0.00 -> 77.1 mm, vias 0 -> 2
- net /INTERFACE/SDA: track 0.00 -> 75.7 mm, vias 0 -> 2
- net /INTERFACE/BUTTON5: track 0.00 -> 74.6 mm
- net /MCU/SPI_LCD_CS: track 0.00 -> 74.3 mm, vias 0 -> 1
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- added copper zone on In2.Cu, net +3V3
- added copper zone on In1.Cu, net GND
Other:
- outline, holes or cut-outs redrawn
- board text added: "Controller Rev 1 Avi Cahoon Isabella Schneider Dexter Siu"
- board text added: "EINK DISPLAY HERE"

Commit message: controller updates
Parts:
- removed D6: LED-G, LED_SMD:LED_0603_1608Metric_Pad1.05x0.95mm_HandSolder
- removed the R11 at (105.7, 126.0)
- removed S7: PRT-14460, samacsys:PRT14460
- added J9: Conn_01x04, Connector_PinHeader_2.54mm:PinHeader_1x04_P2.54mm_Horizontal, F.Cu at (64.5, 119.0)
- added R1: 0, Resistor_SMD:R_0603_1608Metric_Pad0.98x0.95mm_HandSolder, B.Cu at (188.6, 128.5)
- added R12: 10k, Resistor_SMD:R_0603_1608Metric_Pad0.98x0.95mm_HandSolder, B.Cu at (68.9, 111.0)
- added R48: 0, Resistor_SMD:R_0603_1608Metric_Pad0.98x0.95mm_HandSolder, B.Cu at (209.0, 129.2)
- added R49: 0, Resistor_SMD:R_0603_1608Metric_Pad0.98x0.95mm_HandSolder, B.Cu at (207.5, 129.2)
- added TP10: TestPoint, TestPoint:TestPoint_Pad_D3.0mm, F.Cu at (223.2, 124.4)
- added TP11: TestPoint, TestPoint:TestPoint_Pad_D3.0mm, F.Cu at (217.9, 102.3)
- added TP12: TestPoint, TestPoint:TestPoint_Pad_D3.0mm, F.Cu at (75.7, 153.9)
- added TP13: TestPoint, TestPoint:TestPoint_Pad_D3.0mm, F.Cu at (66.4, 184.6)
- added TP14: TestPoint, TestPoint:TestPoint_Pad_D3.0mm, F.Cu at (182.8, 126.9)
- added TP15: TestPoint, TestPoint:TestPoint_Pad_D3.0mm, F.Cu at (95.1, 140.3)
- added TP16: TestPoint, TestPoint:TestPoint_Pad_D3.0mm, F.Cu at (59.3, 153.5)
- C19, C21, C37, C41: value 100nF -> 100n
- D1, D2, D3, TP1, TP2: moved to F.Cu
- L3, L4: footprint parts-lib:CDRH5D18 -> Inductor_SMD:L_0603_1608Metric
- R32: renamed from R31; value 800k -> 787K
- R35: renamed from R34; value DNP -> 0
- R37: renamed from R36; value DNP -> 0
- R7: renamed from R6; moved to F.Cu
- R8: renamed from R7; moved to F.Cu
- R9: renamed from R8; moved to F.Cu
- moved D1 112.4 mm to (188.1, 183.4)
- moved D2 109.3 mm to (186.5, 183.4)
- moved R8 109.1 mm to (186.5, 186.8)
- moved R9 107.9 mm to (188.0, 186.8)
- moved D3 38.2 mm to (114.0, 140.0)
- moved R7 34.8 mm to (116.3, 140.0), turned to 90 degrees
- moved R11 33.2 mm to (131.9, 140.0)
- moved D5 29.8 mm to (130.0, 140.0)
- moved R26 10.5 mm to (69.1, 116.5)
- moved TP7 10.1 mm to (99.7, 140.1)
- moved TP6 6.69 mm to (106.7, 140.6)
- moved C42 5.70 mm to (211.2, 123.7), turned to 180 degrees
- moved C43 5.61 mm to (205.6, 123.8), turned to 0 degrees
- moved L3 3.00 mm to (210.3, 116.9)
- moved TP1 0.99 mm to (222.0, 98.1), turned to 0 degrees
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- renumbered C4 to C10, C13 to C12, C12 to C13, C5 to C2, C7 to C3, C3 to C4, C9 to C5, C10 to C7, C2 to C9, H5 to H1, H1 to H2, H6 to H3, H2 to H4, H7 to H5, H3 to H6, H8 to H7, H4 to H8, R9 to R10, R10 to R11, R12 to R13, R13 to R14, R14 to R15, R15 to R16, R16 to R17, R17 to R18, R18 to R19, R1 to R2, R19 to R20, R20 to R21, R21 to R22, R22 to R23, R23 to R24, R24 to R25, R25 to R26, R26 to R27, R27 to R28, R28 to R29, R2 to R3, R29 to R30, R30 to R31, R32 to R33, R33 to R34, R35 to R36, R37 to R38, R38 to R39, R3 to R4, R39 to R40, R40 to R41, R41 to R42, R42 to R43, R43 to R44, R44 to R45, R45 to R46, R46 to R47, R4 to R5, R5 to R6
Connections:
- net /MCU/LED_DEBUG_R renamed /MCU/LED_NFC_WORKING
- C10 pad 2: +3V3 -> VDD_NFC
- C11 pad 2: +3V3 -> VDD_NFC
- C12 pad 2: +3V3 -> VDD_NFC
- C13 pad 2: +3V3 -> VDD_NFC
- C14 pad 2: +3V3 -> VDD_NFC
- C43 pad 4: Net-(C42-PORT2) -> Net-(C43-PORT2)
- C48 pad 1: Net-(C42-PORT2) -> Net-(C43-PORT2)
- C51 pad 2: Net-(C42-PORT2) -> Net-(C43-PORT2)
- C53 pad 1: Net-(C42-PORT2) -> Net-(C43-PORT2)
- C9 pad 2: +3V3 -> VDD_NFC
- D1 pad 2: /MCU/LED_DEBUG_G -> /MCU/LED_NFC_DONE
- IC1 pad 1: +3V3 -> VDD_NFC
- IC1 pad 10: +3V3 -> VDD_NFC
- IC1 pad 8: +3V3 -> VDD_NFC
- J2 pad 1: /MCU/LED_DEBUG_G -> /MCU/LED_DEBUG_B
- J2 pad 3: /MCU/LED_DEBUG_B -> /MCU/LED_NFC_DONE
- LS1 pad 1: (no net) -> GND
- R2 pad 1: +3V3 -> VDD_NFC
- R3 pad 2: +3V3 -> VDD_NFC
- R46 pad 1: Net-(C42-PORT2) -> Net-(C43-PORT2)
- R5 pad 2: +3V3 -> VDD_NFC
- R7 pad 1: Net-(D1-K) -> Net-(D3-K)
- R9 pad 1: Net-(D3-K) -> Net-(D1-K)
- U1 pad 3: /MCU/LED_DEBUG_G -> /MCU/LED_DEBUG_B
- U1 pad 33: /MCU/LED_DISPLAY_G -> /MCU/PWR_INDICATOR
- U1 pad 5: /MCU/LED_DEBUG_B -> /MCU/LED_NFC_DONE
Routing:
- net /NFC/ANTENNA/ANTENNA_COIL: track 0.00 -> 605.4 mm, vias 0 -> 2
- net /MCU/LED_NFC_DONE: track 0.00 -> 141.4 mm, vias 0 -> 3
- net /MCU/LED_NFC_WORKING: track 64.9 -> 136.0 mm
- net /MCU/PWR_INDICATOR: track 0.00 -> 67.2 mm, vias 0 -> 1
- net /MCU/LED_DEBUG_G: track 56.0 -> 0.00 mm, vias 1 -> 0
- net /MCU/LED_DISPLAY_G: track 27.3 -> 0.00 mm, vias 1 -> 0
- net VDD_NFC: track 0.00 -> 21.7 mm, vias 0 -> 11
- net Net-(C43-PORT2): track 0.00 -> 19.6 mm
- net /INTERFACE/BUSY: track 73.6 -> 91.4 mm, vias 0 -> 1
- net +3V3: track 45.9 -> 30.3 mm, vias 23 -> 15
- net /MCU/LED_DEBUG_B: track 73.9 -> 63.2 mm, vias 1 -> 2
- net /MCU/LED_DISPLAY_R: track 27.4 -> 19.7 mm
- net /INTERFACE/RES#: track 73.2 -> 79.6 mm
- net Net-(C42-PORT1): track 16.9 -> 23.1 mm, vias 0 -> 2
- net GND: track 119.1 -> 125.3 mm, vias 75 -> 77
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- added copper zone on In2.Cu, net VDD_NFC
