File: Ecardz-Controller/Ecardz-Controller.kicad_pcb (KiCad board)
At the start: 4 copper layers, 189 x 115 mm, 186 parts, among them IC1 ST25R3916B-AQWT, IC2 INA180A2IDBVR, J1 MEM2061-01-188-00-A, J10 Conn_01x02, J11 Conn_01x02, J2 Conn_01x04, J3 Conn_01x05, J4 Conn_01x09, J5 Conn_01x01, J6 Conn_01x24, J7 Conn_01x02, J8 Conn_01x04, J9 Conn_01x04, Q1 NMOS, Q2 TMBT3904,LM, U1 STM32G0C1RETx, U2 TPS62160DSG, U3 MIC5504-3.3YM5, U4 CP2110-F02-GM1, Y1 XRCGB27M120F3M00R0

Commit message: turned flex connector around
Parts:
- removed VPP: TestPoint, TestPoint:TestPoint_Pad_D3.0mm
- added TP3: TestPoint, TestPoint:TestPoint_Pad_D3.0mm, F.Cu at (66.4, 192.1)
- D1: renamed from NFC DONE
- D2: renamed from NFC WORKING
- TP10: renamed from VDD NFC
- TP12: renamed from EINK BUSY
- moved C32 19.6 mm to (74.7, 190.1)
- moved R28 18.9 mm to (74.8, 170.9)
- moved C24 16.1 mm to (74.7, 188.4)
- moved R27 15.4 mm to (74.8, 172.9)
- moved D10 13.2 mm to (83.2, 184.7)
- moved D9 13.2 mm to (83.2, 187.2)
- moved C31 13.2 mm to (74.7, 186.9)
- moved L1 13.0 mm to (90.9, 185.5)
- moved C26 11.9 mm to (74.8, 174.4)
- moved C25 11.8 mm to (89.0, 172.3)
- moved D11 11.8 mm to (91.0, 172.3)
- moved Q1 11.8 mm to (86.0, 172.2), turned to 180 degrees
- moved TP13 11.5 mm to (73.2, 193.9)
- moved C23 9.65 mm to (74.7, 185.1)
- moved C27 8.97 mm to (74.7, 175.9)
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- renumbered RX to D7, TX to D8, TAD2 to TP1, BUSY to TP11, BUSY to TP14, 5V_USBC to TP15, GND to TP16, TAD1 to TP2, VIN_PROT to TP4, PGOOD to TP5, FB to TP6, VOS to TP7, SUSPEND to TP8, SUSPEND\ to TP9
Routing:
- net /INTERFACE/RES#: track 91.2 -> 105.1 mm, vias 2 -> 3
- net /INTERFACE/BUSY: track 86.7 -> 79.3 mm, vias 3 -> 4
- net Net-(D9-A): track 21.3 -> 25.7 mm
- net Net-(D10-K): track 21.9 -> 17.7 mm
- net /INTERFACE/SDA: track 81.3 -> 84.7 mm
- net /INTERFACE/VGL: track 16.2 -> 19.2 mm
- net /INTERFACE/VSH2: track 7.46 -> 5.42 mm
- net /INTERFACE/BS1: track 8.88 -> 6.92 mm
- net GND: track 155.6 -> 157.6 mm, vias 106 -> 107
- net /INTERFACE/VCOM: track 8.74 -> 6.88 mm
- net /INTERFACE/D/C#: track 84.3 -> 82.4 mm
- net /INTERFACE/VGH: track 15.7 -> 14.0 mm
- net /INTERFACE/RESE: track 19.5 -> 21.1 mm
- net /INTERFACE/VSH1: track 6.95 -> 5.39 mm
- net /INTERFACE/CS#: track 83.3 -> 81.8 mm
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