File: Ecardz-Controller/POWER.kicad_sch (KiCad schematic)
At the start: 22 parts, among them J1 Conn_01x02, U1 TPS62160DSG, U5 MIC5504-3.3YM5

Commit message: initial work on controller layout
Parts:
- J7: renamed from J1; footprint (none) -> Connector_PinHeader_2.54mm:PinHeader_1x02_P2.54mm_Vertical
- renumbered C1 to C33, C2 to C34, C22 to C35, C23 to C36, D2 to D12, D1 to D13, L1 to L2, R4 to R30, R1 to R31, R2 to R32, R3 to R33, R33 to R34, R31 to R35, R32 to R36, R34 to R37, TP3 to TP4, TP1 to TP5, TP2 to TP6, TP4 to TP7, U1 to U2, U5 to U3
Changed lines of the file:
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@@
 		(dnp no)
 		(fields_autoplaced yes)
-		(property "Reference" "C1"
+		(property "Reference" "C33"
 			(at 87.63 67.3099 0)
 			(effects
@@
 			(project "Ecardz-Controller"
 				(path "/74270717-a116-451e-ac88-5a07ab66056e/686e621e-6f68-4fb8-9509-95408ee4dcf7"
-					(reference "C1")
+					(reference "C33")
 					(unit 1)
 				)
@@
 		(on_board yes)
 		(dnp no)
-		(property "Reference" "R34"
+		(property "Reference" "R37"
 			(at 202.692 66.04 90)
 			(effects
@@
 			(project "Ecardz-Controller"
 				(path "/74270717-a116-451e-ac88-5a07ab66056e/686e621e-6f68-4fb8-9509-95408ee4dcf7"
-					(reference "R34")
+					(reference "R37")
 					(unit 1)
 				)
@@
 		(dnp no)
 		(fields_autoplaced yes)
-		(property "Reference" "C2"
+		(property "Reference" "C34"
 			(at 179.07 67.3099 0)
 			(effects
@@
 			(project "Ecardz-Controller"
 				(path "/74270717-a116-451e-ac88-5a07ab66056e/686e621e-6f68-4fb8-9509-95408ee4dcf7"
-					(reference "C2")
+					(reference "C34")
 					(unit 1)
 				)
@@
 		(dnp no)
 		(fields_autoplaced yes)
-		(property "Reference" "R31"
+		(property "Reference" "R35"
 			(at 186.69 52.07 90)
 			(effects
@@
 			(project "Ecardz-Controller"
 				(path "/74270717-a116-451e-ac88-5a07ab66056e/686e621e-6f68-4fb8-9509-95408ee4dcf7"
-					(reference "R31")
+					(reference "R35")
 					(unit 1)
 				)
@@
 		(dnp no)
 		(fields_autoplaced yes)
-		(property "Reference" "U1"
+		(property "Reference" "U2"
 			(at 124.46 50.8 0)
 			(effects
@@
 			(project "Ecardz-Controller"
 				(path "/74270717-a116-451e-ac88-5a07ab66056e/686e621e-6f68-4fb8-9509-95408ee4dcf7"
-					(reference "U1")
+					(reference "U2")
 					(unit 1)
 				)
@@
 		(dnp no)
 		(fields_autoplaced yes)
-		(property "Reference" "TP3"
+		(property "Reference" "TP4"
 			(at 78.74 53.8479 0)
 			(effects
@@
 			(project "Ecardz-Controller"
 				(path "/74270717-a116-451e-ac88-5a07ab66056e/686e621e-6f68-4fb8-9509-95408ee4dcf7"
-					(reference "TP3")
+					(reference "TP4")
 					(unit 1)
 				)
@@
 		(dnp no)
 		(fields_autoplaced yes)
-		(property "Reference" "#PWR03"
+		(property "Reference" "#PWR045"
 			(at 234.95 57.15 0)
 			(effects
@@
 			(project "Ecardz-Controller"
 				(path "/74270717-a116-451e-ac88-5a07ab66056e/686e621e-6f68-4fb8-9509-95408ee4dcf7"
-					(reference "#PWR03")
+					(reference "#PWR045")
 					(unit 1)
 				)
@@
 		(dnp no)
 		(fields_autoplaced yes)
-		(property "Reference" "D1"
+		(property "Reference" "D13"
 			(at 59.69 52.07 0)
 			(effects
@@
 			(project "Ecardz-Controller"
 				(path "/74270717-a116-451e-ac88-5a07ab66056e/686e621e-6f68-4fb8-9509-95408ee4dcf7"
-					(reference "D1")
+					(reference "D13")
 					(unit 1)
 				)
@@
 		(dnp no)
 		(fields_autoplaced yes)
-		(property "Reference" "#PWR01"
+		(property "Reference" "#PWR042"
 			(at 45.72 90.17 0)
 			(effects
@@
 			(project "Ecardz-Controller"
 				(path "/74270717-a116-451e-ac88-5a07ab66056e/686e621e-6f68-4fb8-9509-95408ee4dcf7"
-					(reference "#PWR01")
+					(reference "#PWR042")
 					(unit 1)
 				)
@@
 		(dnp no)
 		(fields_autoplaced yes)
-		(property "Reference" "R33"
+		(property "Reference" "R34"
 			(at 175.26 40.64 90)
 			(effects
@@
 			(project "Ecardz-Controller"
 				(path "/74270717-a116-451e-ac88-5a07ab66056e/686e621e-6f68-4fb8-9509-95408ee4dcf7"
-					(reference "R33")
+					(reference "R34")
 					(unit 1)
 				)
@@
 		(dnp no)
 		(fields_autoplaced yes)
-		(property "Reference" "#PWR02"
+		(property "Reference" "#PWR043"
 			(at 135.89 90.17 0)
 			(effects
@@
 			(project "Ecardz-Controller"
 				(path "/74270717-a116-451e-ac88-5a07ab66056e/686e621e-6f68-4fb8-9509-95408ee4dcf7"
-					(reference "#PWR02")
+					(reference "#PWR043")
 					(unit 1)
 				)
@@
 		(on_board yes)
 		(dnp no)
-		(property "Reference" "C22"
+		(property "Reference" "C35"
 			(at 193.04 63.246 0)
 			(effects
@@
 			(project "Ecardz-Controller"
 				(path "/74270717-a116-451e-ac88-5a07ab66056e/686e621e-6f68-4fb8-9509-95408ee4dcf7"
-					(reference "C22")
+					(reference "C35")
 					(unit 1)
 				)
@@
 		(dnp no)
 		(fields_autoplaced yes)
-		(property "Reference" "TP4"
+		(property "Reference" "TP7"
 			(at 168.91 53.8479 0)
 			(effects
@@
 			(project "Ecardz-Controller"
 				(path "/74270717-a116-451e-ac88-5a07ab66056e/686e621e-6f68-4fb8-9509-95408ee4dcf7"
-					(reference "TP4")
+					(reference "TP7")
 					(unit 1)
 				)
@@
 		(dnp no)
 		(fields_autoplaced yes)
-		(property "Reference" "R1"
+		(property "Reference" "R31"
 			(at 154.94 60.9599 0)
 			(effects
@@
 			(project "Ecardz-Controller"
 				(path "/74270717-a116-451e-ac88-5a07ab66056e/686e621e-6f68-4fb8-9509-95408ee4dcf7"
-					(reference "R1")
+					(reference "R31")
 					(unit 1)
 				)
@@
 		(dnp no)
 		(fields_autoplaced yes)
-		(property "Reference" "TP1"
+		(property "Reference" "TP5"
 			(at 133.35 38.6079 0)
 			(effects
@@
 			(project "Ecardz-Controller"
 				(path "/74270717-a116-451e-ac88-5a07ab66056e/686e621e-6f68-4fb8-9509-95408ee4dcf7"
-					(reference "TP1")
+					(reference "TP5")
 					(unit 1)
 				)
@@
 		(dnp no)
 		(fields_autoplaced yes)
-		(property "Reference" "R2"
+		(property "Reference" "R32"
 			(at 154.94 72.3899 0)
 			(effects
@@
 			(project "Ecardz-Controller"
 				(path "/74270717-a116-451e-ac88-5a07ab66056e/686e621e-6f68-4fb8-9509-95408ee4dcf7"
-					(reference "R2")
+					(reference "R32")
 					(unit 1)
 				)
@@
 		(dnp no)
 		(fields_autoplaced yes)
-		(property "Reference" "TP2"
+		(property "Reference" "TP6"
 			(at 140.97 64.0079 0)
 			(effects
@@
 			(project "Ecardz-Controller"
 				(path "/74270717-a116-451e-ac88-5a07ab66056e/686e621e-6f68-4fb8-9509-95408ee4dcf7"
-					(reference "TP2")
+					(reference "TP6")
 					(unit 1)
 				)
@@
 		(dnp no)
 		(fields_autoplaced yes)
-		(property "Reference" "#PWR025"
+		(property "Reference" "#PWR044"
 			(at 168.91 46.99 0)
 			(effects
@@
 			(project "Ecardz-Controller"
 				(path "/74270717-a116-451e-ac88-5a07ab66056e/686e621e-6f68-4fb8-9509-95408ee4dcf7"
-					(reference "#PWR025")
+					(reference "#PWR044")
 					(unit 1)
 				)
@@
 		(on_board yes)
 		(dnp no)
-		(property "Reference" "C23"
+		(property "Reference" "C36"
 			(at 236.22 61.976 0)
 			(effects
@@
 			(project "Ecardz-Controller"
 				(path "/74270717-a116-451e-ac88-5a07ab66056e/686e621e-6f68-4fb8-9509-95408ee4dcf7"
-					(reference "C23")
+					(reference "C36")
 					(unit 1)
 				)
@@
 		(dnp no)
 		(fields_autoplaced yes)
-		(property "Reference" "D2"
+		(property "Reference" "D12"
 			(at 59.69 36.83 0)
 			(effects
@@
 			(project "Ecardz-Controller"
 				(path "/74270717-a116-451e-ac88-5a07ab66056e/686e621e-6f68-4fb8-9509-95408ee4dcf7"
-					(reference "D2")
+					(reference "D12")
 					(unit 1)
 				)
@@
 		(dnp no)
 		(fields_autoplaced yes)
-		(property "Reference" "U5"
+		(property "Reference" "U3"
 			(at 217.17 50.8 0)
 			(effects
@@
 			(project "Ecardz-Controller"
 				(path "/74270717-a116-451e-ac88-5a07ab66056e/686e621e-6f68-4fb8-9509-95408ee4dcf7"
-					(reference "U5")
+					(reference "U3")
 					(unit 1)
 				)
@@
 		(dnp no)
 		(fields_autoplaced yes)
-		(property "Reference" "R3"
+		(property "Reference" "R33"
 			(at 161.29 48.2599 0)
 			(effects
@@
 			(project "Ecardz-Controller"
 				(path "/74270717-a116-451e-ac88-5a07ab66056e/686e621e-6f68-4fb8-9509-95408ee4dcf7"
-					(reference "R3")
+					(reference "R33")
 					(unit 1)
 				)
@@
 		(on_board yes)
 		(dnp no)
-		(property "Reference" "J1"
+		(property "Reference" "J7"
 			(at 36.83 58.4199 0)
 			(effects
@@
 			)
 		)
-		(property "Footprint" ""
+		(property "Footprint" "Connector_PinHeader_2.54mm:PinHeader_1x02_P2.54mm_Vertical"
 			(at 39.37 58.42 0)
 			(effects
@@
 			(project "Ecardz-Controller"
 				(path "/74270717-a116-451e-ac88-5a07ab66056e/686e621e-6f68-4fb8-9509-95408ee4dcf7"
-					(reference "J1")
+					(reference "J7")
 					(unit 1)
 				)
@@
 		(on_board yes)
 		(dnp no)
-		(property "Reference" "R4"
+		(property "Reference" "R30"
 			(at 101.346 63.5 90)
 			(effects
@@
 			(project "Ecardz-Controller"
 				(path "/74270717-a116-451e-ac88-5a07ab66056e/686e621e-6f68-4fb8-9509-95408ee4dcf7"
-					(reference "R4")
+					(reference "R30")
 					(unit 1)
 				)
@@
 		(dnp no)
 		(fields_autoplaced yes)
-		(property "Reference" "R32"
+		(property "Reference" "R36"
 			(at 190.5 27.94 90)
 			(effects
@@
 			(project "Ecardz-Controller"
 				(path "/74270717-a116-451e-ac88-5a07ab66056e/686e621e-6f68-4fb8-9509-95408ee4dcf7"
-					(reference "R32")
+					(reference "R36")
 					(unit 1)
 				)
@@
 		(dnp no)
 		(fields_autoplaced yes)
-		(property "Reference" "L1"
+		(property "Reference" "L2"
 			(at 142.24 53.34 90)
 			(effects
@@
 			(project "Ecardz-Controller"
 				(path "/74270717-a116-451e-ac88-5a07ab66056e/686e621e-6f68-4fb8-9509-95408ee4dcf7"
-					(reference "L1")
-					(unit 1)
-				)
+					(reference "L2")
+					(unit 1)
+				)

Commit message: did bulk of controller layout apart from the antenna, added some NCs and other minor clean ups on schematic
Parts:
- L2: footprint SamacSys_Parts:VLS2016 -> samacsys:VLS2016
- R30, R33: footprint (none) -> Resistor_SMD:R_0603_1608Metric_Pad0.98x0.95mm_HandSolder
Changed lines of the file:
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@@
 			)
 		)
-		(property "Footprint" ""
+		(property "Footprint" "Resistor_SMD:R_0603_1608Metric_Pad0.98x0.95mm_HandSolder"
 			(at 159.766 49.784 90)
 			(effects
@@
 			)
 		)
-		(property "Footprint" ""
+		(property "Footprint" "Resistor_SMD:R_0603_1608Metric_Pad0.98x0.95mm_HandSolder"
 			(at 101.346 61.976 90)
 			(effects
@@
 			)
 		)
-		(property "Footprint" "SamacSys_Parts:VLS2016"
+		(property "Footprint" "samacsys:VLS2016"
 			(at 142.24 58.42 0)
 			(effects

Commit message: controller updates
Parts:
- C33: Part Number C0805C105K3RAC3124 -> GRM21BR61C106KE15K
- D12, D13: Part Number (none) -> RB521S30T1G
- J7: Part Number (none) -> 61300211121
- R31: renamed from R30; Part Number (none) -> RC0603FR-07100KL
- R32: renamed from R31; value 800k -> 787K
- R34: renamed from R33; Part Number (none) -> RC0603FR-07100KL
- R35: renamed from R34; value DNP -> 0; Part Number (none) -> RMCF0603ZT0R00; now not fitted
- R36: renamed from R35; Part Number (none) -> RMCF0603ZT0R00
- R37: renamed from R36; value DNP -> 0; Part Number (none) -> RMCF0603ZT0R00; now not fitted
- R38: renamed from R37; Part Number (none) -> RMCF0603ZT0R00
- renumbered R32 to R33

Commit message: updates based on review
Parts:
- added J10: Conn_01x02, Connector_PinHeader_2.54mm:PinHeader_1x02_P2.54mm_Vertical, symbol Connector_Generic:Conn_01x02
Connections:
- net +3V3: now also J10.2 (Pin_2)
- net GND: now also J10.1 (Pin_1)
Other:
- note added: "Alternative Wired Power Source for Card"

Commit message: changed headers to 90 degree angled headers
Parts:
- J10, J7: footprint Connector_PinHeader_2.54mm:PinHeader_1x02_P2.54mm_Vertical -> Connector_PinHeader_2.54mm:PinHeader_1x02_P2.54mm_Horizontal
Changed lines of the file:
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@@
 			)
 		)
-		(property "Footprint" "Connector_PinHeader_2.54mm:PinHeader_1x02_P2.54mm_Vertical"
+		(property "Footprint" "Connector_PinHeader_2.54mm:PinHeader_1x02_P2.54mm_Horizontal"
 			(at 39.37 58.42 0)
 			(effects
@@
 			)
 		)
-		(property "Footprint" "Connector_PinHeader_2.54mm:PinHeader_1x02_P2.54mm_Vertical"
+		(property "Footprint" "Connector_PinHeader_2.54mm:PinHeader_1x02_P2.54mm_Horizontal"
 			(at 88.9 158.75 0)
 			(effects
