File: Ecardz-Controller/antenna.kicad_sch (KiCad schematic)
At the start: 21 parts

Commit message: initial work on controller layout
Parts:
- renumbered C35 to C42, C36 to C43, C34 to C44, C23 to C45, C24 to C46, C25 to C47, C26 to C48, C31 to C49, C32 to C50, C29 to C51, C30 to C52, C27 to C53, R31 to R40, R32 to R41, R27 to R42, R30 to R43, R28 to R44, R24 to R45, R29 to R46
Changed lines of the file:
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@@
 		(dnp yes)
 		(fields_autoplaced yes)
-		(property "Reference" "R32"
+		(property "Reference" "R41"
 			(at 114.3 132.08 90)
 			(effects
@@
 			(project "Ecardz-Controller"
 				(path "/74270717-a116-451e-ac88-5a07ab66056e/414d1147-8205-4839-9169-5f8f29a4e15a/3b8422e5-15b3-4119-8716-a8aee757ed8b"
-					(reference "R32")
+					(reference "R41")
 					(unit 1)
 				)
@@
 		(dnp yes)
 		(fields_autoplaced yes)
-		(property "Reference" "C35"
+		(property "Reference" "C42"
 			(at 86.36 22.86 0)
 			(effects
@@
 			(project "Ecardz-Controller"
 				(path "/74270717-a116-451e-ac88-5a07ab66056e/414d1147-8205-4839-9169-5f8f29a4e15a/3b8422e5-15b3-4119-8716-a8aee757ed8b"
-					(reference "C35")
+					(reference "C42")
 					(unit 1)
 				)
@@
 		(on_board yes)
 		(dnp no)
-		(property "Reference" "C23"
+		(property "Reference" "C45"
 			(at 110.744 65.278 0)
 			(effects
@@
 			(project "Ecardz-Controller"
 				(path "/74270717-a116-451e-ac88-5a07ab66056e/414d1147-8205-4839-9169-5f8f29a4e15a/3b8422e5-15b3-4119-8716-a8aee757ed8b"
-					(reference "C23")
+					(reference "C45")
 					(unit 1)
 				)
@@
 		(dnp no)
 		(fields_autoplaced yes)
-		(property "Reference" "#PWR038"
+		(property "Reference" "#PWR051"
 			(at 60.96 177.8 0)
 			(effects
@@
 			(project "Ecardz-Controller"
 				(path "/74270717-a116-451e-ac88-5a07ab66056e/414d1147-8205-4839-9169-5f8f29a4e15a/3b8422e5-15b3-4119-8716-a8aee757ed8b"
-					(reference "#PWR038")
+					(reference "#PWR051")
 					(unit 1)
 				)
@@
 		(dnp no)
 		(fields_autoplaced yes)
-		(property "Reference" "#PWR034"
+		(property "Reference" "#PWR052"
 			(at 62.23 152.4 0)
 			(effects
@@
 			(project "Ecardz-Controller"
 				(path "/74270717-a116-451e-ac88-5a07ab66056e/414d1147-8205-4839-9169-5f8f29a4e15a/3b8422e5-15b3-4119-8716-a8aee757ed8b"
-					(reference "#PWR034")
+					(reference "#PWR052")
 					(unit 1)
 				)
@@
 		(on_board yes)
 		(dnp no)
-		(property "Reference" "C26"
+		(property "Reference" "C48"
 			(at 141.478 87.376 0)
 			(effects
@@
 			(project "Ecardz-Controller"
 				(path "/74270717-a116-451e-ac88-5a07ab66056e/414d1147-8205-4839-9169-5f8f29a4e15a/3b8422e5-15b3-4119-8716-a8aee757ed8b"
-					(reference "C26")
+					(reference "C48")
 					(unit 1)
 				)
@@
 		(on_board yes)
 		(dnp no)
-		(property "Reference" "C32"
+		(property "Reference" "C50"
 			(at 161.544 50.038 0)
 			(effects
@@
 			(project "Ecardz-Controller"
 				(path "/74270717-a116-451e-ac88-5a07ab66056e/414d1147-8205-4839-9169-5f8f29a4e15a/3b8422e5-15b3-4119-8716-a8aee757ed8b"
-					(reference "C32")
+					(reference "C50")
 					(unit 1)
 				)
@@
 		(dnp yes)
 		(fields_autoplaced yes)
-		(property "Reference" "R31"
+		(property "Reference" "R40"
 			(at 110.49 24.13 90)
 			(effects
@@
 			(project "Ecardz-Controller"
 				(path "/74270717-a116-451e-ac88-5a07ab66056e/414d1147-8205-4839-9169-5f8f29a4e15a/3b8422e5-15b3-4119-8716-a8aee757ed8b"
-					(reference "R31")
+					(reference "R40")
 					(unit 1)
 				)
@@
 		(dnp yes)
 		(fields_autoplaced yes)
-		(property "Reference" "R30"
+		(property "Reference" "R43"
 			(at 123.19 162.56 90)
 			(effects
@@
 			(project "Ecardz-Controller"
 				(path "/74270717-a116-451e-ac88-5a07ab66056e/414d1147-8205-4839-9169-5f8f29a4e15a/3b8422e5-15b3-4119-8716-a8aee757ed8b"
-					(reference "R30")
+					(reference "R43")
 					(unit 1)
 				)
@@
 		(dnp yes)
 		(fields_autoplaced yes)
-		(property "Reference" "R24"
+		(property "Reference" "R45"
 			(at 182.88 69.8499 0)
 			(effects
@@
 			(project "Ecardz-Controller"
 				(path "/74270717-a116-451e-ac88-5a07ab66056e/414d1147-8205-4839-9169-5f8f29a4e15a/3b8422e5-15b3-4119-8716-a8aee757ed8b"
-					(reference "R24")
+					(reference "R45")
 					(unit 1)
 				)
@@
 		(dnp yes)
 		(fields_autoplaced yes)
-		(property "Reference" "C36"
+		(property "Reference" "C43"
 			(at 90.17 130.81 0)
 			(effects
@@
 			(project "Ecardz-Controller"
 				(path "/74270717-a116-451e-ac88-5a07ab66056e/414d1147-8205-4839-9169-5f8f29a4e15a/3b8422e5-15b3-4119-8716-a8aee757ed8b"
-					(reference "C36")
+					(reference "C43")
 					(unit 1)
 				)
@@
 		(dnp no)
 		(fields_autoplaced yes)
-		(property "Reference" "#PWR039"
+		(property "Reference" "#PWR056"
 			(at 189.23 38.1 0)
 			(effects
@@
 			(project "Ecardz-Controller"
 				(path "/74270717-a116-451e-ac88-5a07ab66056e/414d1147-8205-4839-9169-5f8f29a4e15a/3b8422e5-15b3-4119-8716-a8aee757ed8b"
-					(reference "#PWR039")
+					(reference "#PWR056")
 					(unit 1)
 				)
@@
 		(on_board yes)
 		(dnp no)
-		(property "Reference" "C24"
+		(property "Reference" "C46"
 			(at 110.744 81.788 0)
 			(effects
@@
 			(project "Ecardz-Controller"
 				(path "/74270717-a116-451e-ac88-5a07ab66056e/414d1147-8205-4839-9169-5f8f29a4e15a/3b8422e5-15b3-4119-8716-a8aee757ed8b"
-					(reference "C24")
+					(reference "C46")
 					(unit 1)
 				)
@@
 		(on_board yes)
 		(dnp no)
-		(property "Reference" "C31"
+		(property "Reference" "C49"
 			(at 161.544 33.528 0)
 			(effects
@@
 			(project "Ecardz-Controller"
 				(path "/74270717-a116-451e-ac88-5a07ab66056e/414d1147-8205-4839-9169-5f8f29a4e15a/3b8422e5-15b3-4119-8716-a8aee757ed8b"
-					(reference "C31")
+					(reference "C49")
 					(unit 1)
 				)
@@
 		(dnp yes)
 		(fields_autoplaced yes)
-		(property "Reference" "C34"
+		(property "Reference" "C44"
 			(at 90.17 154.94 0)
 			(effects
@@
 			(project ""
 				(path "/74270717-a116-451e-ac88-5a07ab66056e/414d1147-8205-4839-9169-5f8f29a4e15a/3b8422e5-15b3-4119-8716-a8aee757ed8b"
-					(reference "C34")
+					(reference "C44")
 					(unit 1)
 				)
@@
 		(on_board yes)
 		(dnp no)
-		(property "Reference" "C29"
+		(property "Reference" "C51"
 			(at 161.544 112.268 0)
 			(effects
@@
 			(project "Ecardz-Controller"
 				(path "/74270717-a116-451e-ac88-5a07ab66056e/414d1147-8205-4839-9169-5f8f29a4e15a/3b8422e5-15b3-4119-8716-a8aee757ed8b"
-					(reference "C29")
+					(reference "C51")
 					(unit 1)
 				)
@@
 		(on_board yes)
 		(dnp no)
-		(property "Reference" "C25"
+		(property "Reference" "C47"
 			(at 141.478 55.626 0)
 			(effects
@@
 			(project "Ecardz-Controller"
 				(path "/74270717-a116-451e-ac88-5a07ab66056e/414d1147-8205-4839-9169-5f8f29a4e15a/3b8422e5-15b3-4119-8716-a8aee757ed8b"
-					(reference "C25")
+					(reference "C47")
 					(unit 1)
 				)
@@
 		(dnp no)
 		(fields_autoplaced yes)
-		(property "Reference" "#PWR040"
+		(property "Reference" "#PWR053"
 			(at 63.5 46.99 0)
 			(effects
@@
 			(project "Ecardz-Controller"
 				(path "/74270717-a116-451e-ac88-5a07ab66056e/414d1147-8205-4839-9169-5f8f29a4e15a/3b8422e5-15b3-4119-8716-a8aee757ed8b"
-					(reference "#PWR040")
+					(reference "#PWR053")
 					(unit 1)
 				)
@@
 		(dnp no)
 		(fields_autoplaced yes)
-		(property "Reference" "R28"
+		(property "Reference" "R44"
 			(at 165.1 175.2599 0)
 			(effects
@@
 			(project "Ecardz-Controller"
 				(path "/74270717-a116-451e-ac88-5a07ab66056e/414d1147-8205-4839-9169-5f8f29a4e15a/3b8422e5-15b3-4119-8716-a8aee757ed8b"
-					(reference "R28")
+					(reference "R44")
 					(unit 1)
 				)
@@
 		(dnp yes)
 		(fields_autoplaced yes)
-		(property "Reference" "R27"
+		(property "Reference" "R42"
 			(at 123.19 152.4 90)
 			(effects
@@
 			(project "Ecardz-Controller"
 				(path "/74270717-a116-451e-ac88-5a07ab66056e/414d1147-8205-4839-9169-5f8f29a4e15a/3b8422e5-15b3-4119-8716-a8aee757ed8b"
-					(reference "R27")
+					(reference "R42")
 					(unit 1)
 				)
@@
 		(on_board yes)
 		(dnp no)
-		(property "Reference" "C27"
+		(property "Reference" "C53"
 			(at 170.434 74.168 0)
 			(effects
@@
 			(project "Ecardz-Controller"
 				(path "/74270717-a116-451e-ac88-5a07ab66056e/414d1147-8205-4839-9169-5f8f29a4e15a/3b8422e5-15b3-4119-8716-a8aee757ed8b"
-					(reference "C27")
+					(reference "C53")
 					(unit 1)
 				)
@@
 		(dnp no)
 		(fields_autoplaced yes)
-		(property "Reference" "#PWR032"
+		(property "Reference" "#PWR054"
 			(at 95.25 80.01 0)
 			(effects
@@
 			(project "Ecardz-Controller"
 				(path "/74270717-a116-451e-ac88-5a07ab66056e/414d1147-8205-4839-9169-5f8f29a4e15a/3b8422e5-15b3-4119-8716-a8aee757ed8b"
-					(reference "#PWR032")
+					(reference "#PWR054")
 					(unit 1)
 				)
@@
 		(dnp no)
 		(fields_autoplaced yes)
-		(property "Reference" "#PWR035"
+		(property "Reference" "#PWR055"
 			(at 162.56 187.96 0)
 			(effects
@@
 			(project "Ecardz-Controller"
 				(path "/74270717-a116-451e-ac88-5a07ab66056e/414d1147-8205-4839-9169-5f8f29a4e15a/3b8422e5-15b3-4119-8716-a8aee757ed8b"
-					(reference "#PWR035")
+					(reference "#PWR055")
 					(unit 1)
 				)
@@
 		(on_board yes)
 		(dnp no)
-		(property "Reference" "C30"
+		(property "Reference" "C52"
 			(at 161.544 128.778 0)
 			(effects
@@
 			(project "Ecardz-Controller"
 				(path "/74270717-a116-451e-ac88-5a07ab66056e/414d1147-8205-4839-9169-5f8f29a4e15a/3b8422e5-15b3-4119-8716-a8aee757ed8b"
-					(reference "C30")
+					(reference "C52")
 					(unit 1)
 				)
@@
 		(dnp no)
 		(fields_autoplaced yes)
-		(property "Reference" "R29"
+		(property "Reference" "R46"
 			(at 191.77 25.3999 0)
 			(effects
@@
 			(project "Ecardz-Controller"
 				(path "/74270717-a116-451e-ac88-5a07ab66056e/414d1147-8205-4839-9169-5f8f29a4e15a/3b8422e5-15b3-4119-8716-a8aee757ed8b"
-					(reference "R29")
-					(unit 1)
-				)
+					(reference "R46")
+					(unit 1)
+				)

Commit message: did bulk of controller layout apart from the antenna, added some NCs and other minor clean ups on schematic
Parts:
- C42, C43, C44: footprint LXRW0YV600054 -> samacsys:LXRW0YV600054
Changed lines of the file:
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@@
 			)
 		)
-		(property "Footprint" "LXRW0YV600054"
+		(property "Footprint" "samacsys:LXRW0YV600054"
 			(at 96.52 125.4 0)
 			(effects
@@
 			)
 		)
-		(property "Footprint" "LXRW0YV600054"
+		(property "Footprint" "samacsys:LXRW0YV600054"
 			(at 100.33 233.35 0)
 			(effects
@@
 			)
 		)
-		(property "Footprint" "LXRW0YV600054"
+		(property "Footprint" "samacsys:LXRW0YV600054"
 			(at 100.33 257.48 0)
 			(effects

Commit message: controller updates
Parts:
- added R48, R49: 0, Resistor_SMD:R_0603_1608Metric_Pad0.98x0.95mm_HandSolder, symbol Device:R_US
- C42, C43, C44: Part Number (none) -> LXRW0YV600-054
- C45, C46: Part Number (none) -> VJ0603Y681KXACW1BC
- C47, C48: Part Number (none) -> CC0603JRNPO0BN181
- C49, C52: Part Number (none) -> CC0603JRNPO9BN820
- C50, C51: Part Number (none) -> C0603C100J5GACTU
- C53: Part Number (none) -> C0603C241G5HACTU
- L3, L4: footprint parts-lib:CDRH5D18 -> Inductor_SMD:L_0603_1608Metric; Part Number (none) -> MLJ1608WR27JT000
- R41: renamed from R40; Part Number (none) -> RMCF0603ZT0R00
- R42: renamed from R41; Part Number (none) -> RMCF0603ZT0R00
- R43: renamed from R42; Part Number (none) -> RMCF0603ZT0R00
- R44: renamed from R43; Part Number (none) -> RMCF0603ZT0R00
- R45: renamed from R44; Part Number (none) -> RMCF0603ZT0R00
- R46: renamed from R45; Part Number (none) -> RMCF0603ZT0R00
- R47: renamed from R46; Part Number (none) -> RMCF0603ZT0R00
Connections:
- net at C42.4 (PORT2), C47.1, C50.1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: now also R48.1; no longer C43.4 (PORT2), C48.1, C51.2, C53.1, R46.1
- new net: C43.4 (PORT2), C48.1, C51.2, C53.1, R46.1, R49.1
- new net ANTENNA_COIL: R48.2, R49.2
Other:
- moved on the sheet: C53, R46
