File: Ecardz-Proto-Rev2/Ecardz-Proto.kicad_sch (KiCad schematic)
At the start: 4 parts

Commit message: Started board layout + antenna
Parts:
- H1, H2, H3, H4: footprint MountingHole:MountingHole_2.5mm_Pad_TopBottom -> MountingHole:MountingHole_2.2mm_M2_DIN965
Changed lines of the file:
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@@
 			)
 		)
-		(property "Footprint" "MountingHole:MountingHole_2.5mm_Pad_TopBottom"
+		(property "Footprint" "MountingHole:MountingHole_2.2mm_M2_DIN965"
 			(at 92.71 19.05 0)
 			(effects
@@
 			)
 		)
-		(property "Footprint" "MountingHole:MountingHole_2.5mm_Pad_TopBottom"
+		(property "Footprint" "MountingHole:MountingHole_2.2mm_M2_DIN965"
 			(at 41.91 19.05 0)
 			(effects
@@
 			)
 		)
-		(property "Footprint" "MountingHole:MountingHole_2.5mm_Pad_TopBottom"
+		(property "Footprint" "MountingHole:MountingHole_2.2mm_M2_DIN965"
 			(at 17.78 19.05 0)
 			(effects
@@
 			)
 		)
-		(property "Footprint" "MountingHole:MountingHole_2.5mm_Pad_TopBottom"
+		(property "Footprint" "MountingHole:MountingHole_2.2mm_M2_DIN965"
 			(at 67.31 19.05 0)
 			(effects

Commit message: final schematic
final schematic done and BOM generated except for pogo pins and capacitors
Other:
- sheet EINK ports: added EINK_POWER_CTRL_N; removed none
- sheet NFC ports: added NFC_POWER; removed none
- sheet STM ports: added EINK_POWER_CTRL_N, NFC_POWER; removed none
Changed lines of the file:
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@@
+	(wire
+		(pts
+			(xy 101.6 91.44) (xy 113.03 91.44)
+		)
+		(stroke
+			(width 0)
+			(type default)
+		)
+	)
 	(wire
 		(pts
@@
 		(pts
 			(xy 101.6 83.82) (xy 113.03 83.82)
+		)
+		(stroke
+			(width 0)
+			(type default)
+		)
+	)
+	(wire
+		(pts
+			(xy 153.67 83.82) (xy 168.91 83.82)
 		)
 		(stroke
@@
 			)
 		)
+		(pin "NFC_POWER" input
+			(at 168.91 83.82 180)
+			(effects
+				(font
+					(size 1.27 1.27)
+				)
+				(justify left)
+			)
+		)
 		(instances
 			(project "Ecardz-Proto"
@@
 		)
 		(pin "TSCL" input
-			(at 101.6 91.44 0)
+			(at 101.6 96.52 0)
 			(effects
 				(font
@@
 		)
 		(pin "TSDA" input
-			(at 101.6 93.98 0)
+			(at 101.6 99.06 0)
 			(effects
 				(font
@@
 		(pin "SPI_EINK_CS#" input
 			(at 101.6 76.2 0)
+			(effects
+				(font
+					(size 1.27 1.27)
+				)
+				(justify right)
+			)
+		)
+		(pin "EINK_POWER_CTRL_N" input
+			(at 101.6 91.44 0)
 			(effects
 				(font
@@
 			)
 		)
+		(pin "NFC_POWER" input
+			(at 153.67 83.82 0)
+			(effects
+				(font
+					(size 1.27 1.27)
+				)
+				(justify right)
+			)
+		)
+		(pin "EINK_POWER_CTRL_N" input
+			(at 113.03 91.44 180)
+			(effects
+				(font
+					(size 1.27 1.27)
+				)
+				(justify left)
+			)
+		)
